File: pcb/relay/relay.kicad_pcb (KiCad board)
At the start: 2 copper layers, 96.5 x 66 mm, 20 parts, among them J1 ScrewTerminal, U1 PinHeader8, U2 PinHeader8

Commit message: realy
Parts:
- added D11: ~, Diode_SMD:D_SOD-123, F.Cu at (71.1, 54.6)
- added D12: ~, Diode_SMD:D_SOD-123, F.Cu at (71.1, 27.9)
- added D13: ~, Diode_SMD:D_SOD-123, F.Cu at (101.6, 33.0)
- added D14: ~, Diode_SMD:D_SOD-123, F.Cu at (118.1, 54.6)
- added Q1: ~, Package_TO_SOT_SMD:SOT-23, F.Cu at (66.0, 47.0)
- added Q2: ~, Package_TO_SOT_SMD:SOT-23, F.Cu at (55.9, 40.6)
- added Q3: ~, Package_TO_SOT_SMD:SOT-23, F.Cu at (66.0, 40.6)
- added Q4: ~, Package_TO_SOT_SMD:SOT-23, F.Cu at (55.9, 47.0)
- added R11: ~, Resistor_SMD:R_0603_1608Metric, F.Cu at (62.2, 45.7)
- added R12: ~, Resistor_SMD:R_0603_1608Metric, F.Cu at (52.1, 39.4)
- added R13: ~, Resistor_SMD:R_0603_1608Metric, F.Cu at (62.2, 39.4)
- added R14: ~, Resistor_SMD:R_0603_1608Metric, F.Cu at (52.1, 45.7)
- moved K3 43.7 mm to (111.8, 33.0), turned to -90 degrees
- moved K2 20.9 mm to (78.7, 33.0), turned to -90 degrees
- moved K1 20.5 mm to (78.7, 58.4), turned to -90 degrees
- moved K4 12.7 mm to (111.8, 58.4), turned to -90 degrees
Connections:
- K1 pad 2: unconnected-(K1-Pad2) -> /5V
- K1 pad 5: unconnected-(K1-Pad5) -> Net-(D11-A)
- K2 pad 2: unconnected-(K2-Pad2) -> /5V
- K2 pad 5: unconnected-(K2-Pad5) -> Net-(D12-A)
- K3 pad 2: unconnected-(K3-Pad2) -> /5V
- K3 pad 5: unconnected-(K3-Pad5) -> Net-(D13-A)
- K4 pad 2: unconnected-(K4-Pad2) -> /5V
- K4 pad 5: unconnected-(K4-Pad5) -> Net-(D14-A)
- U1 pad 2: unconnected-(U1-Pin_2-Pad2) -> Net-(U1-Pin_2)
- U2 pad 1: unconnected-(U2-Pin_1-Pad1) -> Net-(U2-Pin_1)
- U2 pad 2: unconnected-(U2-Pin_2-Pad2) -> Net-(U2-Pin_2)
- U2 pad 4: unconnected-(U2-Pin_4-Pad4) -> Net-(U2-Pin_4)
Routing:
- net /ACL: track 0.00 -> 126.4 mm
- net /5V: track 66.9 -> 190.0 mm, vias 0 -> 1
- net Net-(D14-A): track 0.00 -> 90.6 mm, vias 0 -> 1
- net /ACN: track 0.00 -> 76.2 mm
- net Net-(D13-A): track 0.00 -> 64.5 mm
- net Net-(J3-Pin_4): track 0.00 -> 54.4 mm
- net Net-(D12-A): track 0.00 -> 47.5 mm, vias 0 -> 2
- net Net-(J4-Pin_2): track 0.00 -> 43.0 mm
- net /GND: track 112.2 -> 152.1 mm, vias 0 -> 2
- net Net-(D11-A): track 0.00 -> 28.1 mm, vias 0 -> 1
- net Net-(U2-Pin_4): track 0.00 -> 25.9 mm, vias 0 -> 1
- net Net-(U1-Pin_2): track 0.00 -> 23.9 mm
- net Net-(U2-Pin_1): track 0.00 -> 20.8 mm, vias 0 -> 1
- net Net-(J3-Pin_2): track 0.00 -> 17.3 mm
- net Net-(J4-Pin_4): track 0.00 -> 16.3 mm
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
Commit message: relay update
Parts:
- added REF**: MountingHole_3.2mm_M3, MountingHole:MountingHole_3.2mm_M3, F.Cu at (116.8, 30.5)
- added REF**: MountingHole_3.2mm_M3, MountingHole:MountingHole_3.2mm_M3, F.Cu at (30.5, 86.4)
- added REF**: MountingHole_3.2mm_M3, MountingHole:MountingHole_3.2mm_M3, F.Cu at (116.8, 86.4)
- added REF**: MountingHole_3.2mm_M3, MountingHole:MountingHole_3.2mm_M3, F.Cu at (30.5, 30.5)
- moved D13 2.54 mm to (101.6, 35.6)
- moved D14 2.54 mm to (118.1, 57.1)
- moved K3 2.54 mm to (111.8, 35.6)
- moved K4 2.54 mm to (111.8, 61.0)
Routing:
- net Net-(D13-A): track 64.5 -> 55.5 mm
- net Net-(J4-Pin_2): track 43.0 -> 40.5 mm
- net /ACL: track 126.4 -> 129.0 mm
- net Net-(D14-A): track 90.6 -> 89.5 mm
- net Net-(J4-Pin_4): track 16.3 -> 15.2 mm

Commit message: wip
Parts:
- J1: value ScrewTerminal -> ~
- R1: value ~ -> 4.7k
- R11, R12, R13, R14: value ~ -> 1k
- R4: value ~ -> 330
- U1, U2: value PinHeader8 -> ~
Changed lines of the file:
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@@
 			)
 		)
-		(property "Value" "~"
+		(property "Value" "1k"
 			(at 0 1.43 0)
 			(layer "F.Fab")
@@
 			(fill no)
 			(layer "Cmts.User")
-			(net 108)
 		)
 		(fp_circle
@@
 			(fill no)
 			(layer "F.CrtYd")
-			(net 108)
 		)
 		(fp_text user "${REFERENCE}"
@@
 			)
 		)
-		(property "Value" "PinHeader8"
+		(property "Value" "~"
 			(at 0 20.55 90)
 			(layer "F.Fab")
@@
 			(fill no)
 			(layer "Cmts.User")
-			(net 108)
 		)
 		(fp_circle
@@
 			(fill no)
 			(layer "F.CrtYd")
-			(net 108)
 		)
 		(fp_text user "${REFERENCE}"
@@
 			)
 		)
-		(property "Value" "~"
+		(property "Value" "1k"
 			(at 0 1.43 0)
 			(layer "F.Fab")
@@
 			(fill no)
 			(layer "Cmts.User")
-			(net 108)
 		)
 		(fp_circle
@@
 			(fill no)
 			(layer "F.CrtYd")
-			(net 108)
 		)
 		(fp_text user "${REFERENCE}"
@@
 			)
 		)
-		(property "Value" "PinHeader8"
+		(property "Value" "~"
 			(at 0 20.55 90)
 			(layer "F.Fab")
@@
 			)
 		)
-		(property "Value" "ScrewTerminal"
+		(property "Value" "~"
 			(at 0 1 90)
 			(unlocked yes)
@@
 			(fill no)
 			(layer "Cmts.User")
-			(net 108)
 		)
 		(fp_circle
@@
 			(fill no)
 			(layer "F.CrtYd")
-			(net 108)
 		)
 		(fp_text user "${REFERENCE}"
@@
 			)
 		)
-		(property "Value" "~"
+		(property "Value" "4.7k"
 			(at 0 1.43 0)
 			(layer "F.Fab")
@@
 			)
 		)
+		(property "value" "hello"
+			(at 0 0 180)
+			(unlocked yes)
+			(layer "F.Fab")
+			(hide yes)
+			(effects
+				(font
+					(size 1 1)
+					(thickness 0.15)
+				)
+			)
+		)
 		(property ki_fp_filters "R_*")
 		(sheetname "/")
@@
 			)
 		)
-		(property "Value" "~"
+		(property "Value" "1k"
 			(at 0 1.43 0)
 			(layer "F.Fab")
@@
 			)
 		)
-		(property "Value" "~"
+		(property "Value" "330"
 			(at 0 1.43 0)
 			(layer "F.Fab")
@@
 			)
 		)
-		(property "Value" "~"
+		(property "Value" "1k"
 			(at 0 1.43 0)
 			(layer "F.Fab")
