File: pcb/relay/relay.kicad_sch (KiCad schematic)
At the start: 32 parts, among them J1 ScrewTerminal, U1 PinHeader8, U2 PinHeader8

Commit message: realy
Parts:
- D11, D12, D13, D14: footprint Diode_SMD:D_SMA -> Diode_SMD:D_SOD-123

Commit message: relay update
Parts:
- Q1, Q2, Q3, Q4: lcscRot (none) -> 180
Changed lines of the file:
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@@
+      )
+    )
+    (property "lcscRot" "180"
+      (effects
+        (hide yes)
       )
     )
@@
       )
     )
+    (property "lcscRot" "180"
+      (effects
+        (hide yes)
+      )
+    )
   )
   (symbol
@@
       )
     )
+    (property "lcscRot" "180"
+      (effects
+        (hide yes)
+      )
+    )
   )
   (symbol
@@
       )
     )
+    (property "lcscRot" "180"
+      (effects
+        (hide yes)
+      )
+    )

Commit message: wip
Parts:
- D1, J2, J3, J4, J5, U3, U4, U5, U6, U7, U8: value ~ -> (none)
- J1: value ScrewTerminal -> (none)
- R1: value ~ -> 4.7k; value (none) -> hello
- R11, R12, R13, R14: value (none) -> 1k
- R4: value ~ -> 330
- U1, U2: value PinHeader8 -> (none)
