File: pcb/gpio/gpio.kicad_pcb (KiCad board)
At the start: 2 copper layers, 96.5 x 66 mm, 20 parts, among them J1 ScrewTerminal, U1 PinHeader8, U2 PinHeader8

Commit message: gpio
Connections:
- J2 pad 1: unconnected-(J2-Pin_1-Pad1) -> /GND
- J2 pad 2: unconnected-(J2-Pin_2-Pad2) -> /3V3
- J2 pad 3: unconnected-(J2-Pin_3-Pad3) -> Net-(J2-Pin_3)
- J2 pad 4: unconnected-(J2-Pin_4-Pad4) -> Net-(J2-Pin_4)
- J3 pad 1: unconnected-(J3-Pin_1-Pad1) -> /GND
- J3 pad 2: unconnected-(J3-Pin_2-Pad2) -> /3V3
- J3 pad 3: unconnected-(J3-Pin_3-Pad3) -> Net-(J3-Pin_3)
- J3 pad 4: unconnected-(J3-Pin_4-Pad4) -> Net-(J3-Pin_4)
- J4 pad 1: unconnected-(J4-Pin_1-Pad1) -> Net-(J4-Pin_1)
- J4 pad 2: unconnected-(J4-Pin_2-Pad2) -> Net-(J4-Pin_2)
- J4 pad 3: unconnected-(J4-Pin_3-Pad3) -> Net-(J4-Pin_3)
- J4 pad 4: unconnected-(J4-Pin_4-Pad4) -> Net-(J4-Pin_4)
- U1 pad 2: unconnected-(U1-Pin_2-Pad2) -> Net-(J3-Pin_4)
- U1 pad 3: unconnected-(U1-Pin_3-Pad3) -> Net-(J4-Pin_1)
- U1 pad 6: unconnected-(U1-Pin_6-Pad6) -> Net-(J4-Pin_2)
- U1 pad 7: unconnected-(U1-Pin_7-Pad7) -> Net-(J4-Pin_3)
- U1 pad 8: unconnected-(U1-Pin_8-Pad8) -> Net-(J4-Pin_4)
- U2 pad 1: unconnected-(U2-Pin_1-Pad1) -> Net-(J2-Pin_3)
- U2 pad 2: unconnected-(U2-Pin_2-Pad2) -> Net-(J2-Pin_4)
- U2 pad 4: unconnected-(U2-Pin_4-Pad4) -> Net-(J3-Pin_3)
Routing:
- net Net-(J4-Pin_4): track 0.00 -> 94.6 mm
- net Net-(J4-Pin_1): track 0.00 -> 93.4 mm
- net Net-(J4-Pin_3): track 0.00 -> 90.6 mm
- net Net-(J3-Pin_3): track 0.00 -> 89.3 mm
- net Net-(J3-Pin_4): track 0.00 -> 87.6 mm
- net Net-(J4-Pin_2): track 0.00 -> 86.5 mm
- net Net-(J2-Pin_4): track 0.00 -> 77.4 mm
- net Net-(J2-Pin_3): track 0.00 -> 74.3 mm
- net /3V3: track 48.4 -> 106.0 mm
- net /GND: track 112.2 -> 150.7 mm
- net /CANL: vias 0 -> 1
- net /CANH: vias 0 -> 1

Commit message: gpio pcb fixes
Parts:
- added D11: ~, Diode_SMD:D_0603_1608Metric, F.Cu at (118.1, 55.9)
- added D12: ~, Diode_SMD:D_0603_1608Metric, F.Cu at (118.1, 53.3)
- added D13: ~, Diode_SMD:D_0603_1608Metric, F.Cu at (118.1, 50.8)
- added D14: ~, Diode_SMD:D_0603_1608Metric, F.Cu at (118.1, 48.3)
- added D15: ~, Diode_SMD:D_0603_1608Metric, F.Cu at (118.1, 45.7)
- added D16: ~, Diode_SMD:D_0603_1608Metric, F.Cu at (118.1, 43.2)
- added D17: ~, Diode_SMD:D_0603_1608Metric, F.Cu at (118.1, 40.6)
- added D18: ~, Diode_SMD:D_0603_1608Metric, F.Cu at (118.1, 38.1)
- added R11: 1k, Resistor_SMD:R_0603_1608Metric, F.Cu at (113.0, 55.9)
- added R12: 1k, Resistor_SMD:R_0603_1608Metric, F.Cu at (113.0, 53.3)
- added R13: 1k, Resistor_SMD:R_0603_1608Metric, F.Cu at (113.0, 50.8)
- added R14: 1k, Resistor_SMD:R_0603_1608Metric, F.Cu at (113.0, 48.3)
- added R15: 1k, Resistor_SMD:R_0603_1608Metric, F.Cu at (113.0, 45.7)
- added R16: 1k, Resistor_SMD:R_0603_1608Metric, F.Cu at (113.0, 43.2)
- added R17: 1k, Resistor_SMD:R_0603_1608Metric, F.Cu at (113.0, 40.6)
- added R18: 1k, Resistor_SMD:R_0603_1608Metric, F.Cu at (113.0, 38.1)
- J1: value ScrewTerminal -> ~
- R1: value ~ -> 4.7k
- R4: value ~ -> 330
- U1, U2: value PinHeader8 -> ~
Routing:
- net /GND: track 150.7 -> 240.8 mm, vias 0 -> 1
- net Net-(J3-Pin_4): track 87.6 -> 138.8 mm, vias 0 -> 2
- net Net-(J4-Pin_1): track 93.4 -> 142.1 mm, vias 0 -> 2
- net Net-(J4-Pin_2): track 86.5 -> 132.7 mm, vias 0 -> 2
- net Net-(J4-Pin_3): track 90.6 -> 134.2 mm, vias 0 -> 2
- net Net-(J4-Pin_4): track 94.6 -> 135.7 mm, vias 0 -> 2
- net Net-(J2-Pin_3): track 74.3 -> 115.4 mm, vias 0 -> 1
- net Net-(J2-Pin_4): track 77.4 -> 116.0 mm, vias 0 -> 1
- net Net-(J3-Pin_3): track 89.3 -> 125.3 mm, vias 0 -> 1
- net Net-(D18-A): track 0.00 -> 3.47 mm
- net Net-(D17-A): track 0.00 -> 3.47 mm
- net Net-(D16-A): track 0.00 -> 3.47 mm
- net Net-(D15-A): track 0.00 -> 3.47 mm
- net Net-(D14-A): track 0.00 -> 3.47 mm
- net Net-(D13-A): track 0.00 -> 3.47 mm
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