File: pcb/liu/liu.kicad_pcb (KiCad board)
At the start: 2 copper layers, 96.5 x 66 mm, 18 parts

Commit message: liu
Parts:
- added J6: ~, Connector_PinSocket_2.54mm:PinSocket_1x04_P2.54mm_Vertical, F.Cu at (76.2, 38.1)
- added J7: ~, Connector_PinSocket_2.54mm:PinSocket_1x05_P2.54mm_Vertical, F.Cu at (86.4, 38.1)
Connections:
- U1 pad 2: unconnected-(U1-Pin_2-Pad2) -> Net-(J6-Pin_4)
- U1 pad 3: unconnected-(U1-Pin_3-Pad3) -> Net-(J6-Pin_3)
- U1 pad 6: unconnected-(U1-Pin_6-Pad6) -> Net-(J7-Pin_3)
- U1 pad 7: unconnected-(U1-Pin_7-Pad7) -> Net-(J7-Pin_4)
- U1 pad 8: unconnected-(U1-Pin_8-Pad8) -> Net-(J7-Pin_5)
Routing:
- net Net-(J6-Pin_3): track 0.00 -> 61.6 mm
- net Net-(J6-Pin_4): track 0.00 -> 56.2 mm
- net Net-(J7-Pin_3): track 0.00 -> 53.1 mm
- net /3V3: track 36.8 -> 87.6 mm
- net Net-(J7-Pin_4): track 0.00 -> 49.5 mm
- net Net-(J7-Pin_5): track 0.00 -> 45.9 mm
- net /GND: track 136.6 -> 168.1 mm
- net Net-(U1-Pin_1): track 44.0 -> 49.9 mm

Commit message: pcb
Parts:
- added R5: 1k, Resistor_SMD:R_0603_1608Metric, F.Cu at (54.6, 66.0)
- added R6: 1k, Resistor_SMD:R_0603_1608Metric, F.Cu at (53.3, 68.6)
- added R7: 1k, Resistor_SMD:R_0603_1608Metric, F.Cu at (52.1, 71.1)
- added R8: 1k, Resistor_SMD:R_0603_1608Metric, F.Cu at (50.8, 73.7)
- added R9: 1k, Resistor_SMD:R_0603_1608Metric, F.Cu at (33.0, 73.7)
- added U10: ~, Connector_PinSocket_2.54mm:PinSocket_1x08_P2.54mm_Vertical, F.Cu at (45.7, 63.5)
- added U9: ~, Connector_PinSocket_2.54mm:PinSocket_1x08_P2.54mm_Vertical, F.Cu at (27.9, 78.7)
- R1: value ~ -> 4.7k
- R4: value ~ -> 330
- moved D1 53.3 mm to (81.3, 61.0)
- moved U6 43.3 mm to (94.7, 71.6)
- moved U7 43.3 mm to (94.7, 61.0)
- moved U5 43.3 mm to (76.2, 71.6)
- moved U8 43.3 mm to (76.2, 61.0)
Connections:
- U1 pad 5: unconnected-(U1-Pin_5-Pad5) -> Net-(U1-Pin_5)
- U2 pad 1: unconnected-(U2-Pin_1-Pad1) -> Net-(U2-Pin_1)
- U2 pad 2: unconnected-(U2-Pin_2-Pad2) -> Net-(U2-Pin_2)
- U2 pad 3: unconnected-(U2-Pin_3-Pad3) -> Net-(U2-Pin_3)
- U2 pad 4: unconnected-(U2-Pin_4-Pad4) -> Net-(U2-Pin_4)
Routing:
- net /5V: track 66.9 -> 136.9 mm
- net /GND: track 168.1 -> 227.1 mm
- net Net-(U2-Pin_4): track 0.00 -> 41.5 mm, vias 0 -> 1
- net Net-(U2-Pin_3): track 0.00 -> 38.5 mm, vias 0 -> 1
- net Net-(U2-Pin_2): track 0.00 -> 35.4 mm, vias 0 -> 1
- net Net-(U2-Pin_1): track 0.00 -> 32.3 mm, vias 0 -> 1
- net /12V: track 50.7 -> 79.7 mm
- net Net-(U1-Pin_5): track 0.00 -> 24.1 mm
- net Net-(U10-Pin_4): track 0.00 -> 16.1 mm
- net Net-(U10-Pin_3): track 0.00 -> 13.8 mm
- net /3V3: track 87.6 -> 101.2 mm
- net Net-(U10-Pin_2): track 0.00 -> 11.4 mm
- net Net-(U10-Pin_1): track 0.00 -> 9.12 mm
- net Net-(U9-Pin_5): track 0.00 -> 6.84 mm
